File: PCB/Cody.kicad_sch (KiCad schematic)
At the start: 26 parts, among them J1 Left Encoder, J12 12V Output, J13 Battery Discharge, J14 6V Input, J15 TCS34725 Color Sensor, J16 TCS34725 Color Sensor, J2 Right Encoder, J5 A1 Encoder, J6 A2 Encoder, J7 Battery Balance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

Commit message: 11-03-2026
Parts:
- removed J12: 12V Output, Connector_AMASS:AMASS_XT60-F_1x02_P7.20mm_Vertical, symbol Library:Conn_01x02
- removed J16: TCS34725 Color Sensor, Connector_JST:JST_XH_B7B-XH-A_1x07_P2.50mm_Vertical, symbol Library:Conn_01x07
- removed J8: A3 Servo, Connector_JST:JST_XH_B3B-XH-A_1x03_P2.50mm_Vertical, symbol Library:Conn_01x03
- removed J9: A4 Servo, Connector_JST:JST_XH_B3B-XH-A_1x03_P2.50mm_Vertical, symbol Library:Conn_01x03
- added J3: A3 Encoder, Connector_JST:JST_XH_B6B-XH-A_1x06_P2.50mm_Vertical, symbol Library:Conn_01x06
- added J4: A4 Encoder, Connector_JST:JST_XH_B6B-XH-A_1x06_P2.50mm_Vertical, symbol Library:Conn_01x06
- added J8: Camera, Connector_JST:JST_XH_B2B-XH-A_1x02_P2.50mm_Vertical, symbol Library:Conn_01x02
- added U7: ~, Dependencies:TB6612FNG, symbol Library:TB6612FNG_Breakout
Connections:
- net BMS_IN_4 is gone; now on net GND: J7.4 (Pin_4), R6.2
- net +12V: now also U7.1 (VM)
- net +3V3: now also J3.5 (Pin_5), J4.5 (Pin_5), U7.2 (VCC)
- net A1_A: now also U1.J2-5 (IO34); no longer U1.J3-12 (IO16)
- net A1_B: now also U1.J2-6 (IO35); no longer U1.J3-11 (IO17)
- net A1_PWM: now also U1.J3-12 (IO16); no longer U1.J2-12 (IO14)
- net A2_A: now also U1.J2-3 (SENSOR_VP); no longer U1.J3-9 (IO18)
- net A2_B: now also U1.J2-4 (SENSOR_VN); no longer U1.J3-8 (IO19)
- net A2_PWM: now also U1.J3-11 (IO17); no longer U1.J3-16 (IO15)
- net BUZZER: now also U1.J3-10 (IO5); no longer U6.4 (P13)
- net GND: now also J3.6 (Pin_6), J4.6 (Pin_6), U7.16 (GND), U7.8 (GND); no longer U2.3 (GND), U3.3 (GND)
- net LED_B: now also U6.7 (P16); no longer U6.3 (P12)
- net LED_G: now also U6.6 (P15); no longer U6.2 (P11)
- net LED_R: now also U6.5 (P14); no longer U6.1 (P10)
- net L_PWM: now also U1.J3-15 (IO2); no longer U1.J3-13 (IO4)
- net R_PWM: now also U1.J3-13 (IO4); no longer U1.J3-10 (IO5)
- net STNDBY: now also U6.8 (P17), U7.12 (STNDBY); no longer U1.J3-15 (IO2)
- net A3 renamed A3_A
- net A3_A: now also J3.3 (Pin_3)
- net A4 renamed A3_B
- net A3_B: now also J3.4 (Pin_4)
- net SCL_1 renamed CAM_RX
- net CAM_RX: now also J8.2 (Pin_2)
- net SDA_1 renamed CAM_TX
- net CAM_TX: now also J8.1 (Pin_1)
- new net A3_IN_1: U6.1 (P10), U7.11 (AIN1)
- new net A3_IN_2: U6.2 (P11), U7.10 (AIN2)
- new net A3_OUT_1: J3.1 (Pin_1), U7.4 (AO1)
- new net A3_OUT_2: J3.2 (Pin_2), U7.5 (AO2)
- new net A3_PWM: U1.J3-9 (IO18), U7.9 (PWMA)
- new net A4_A: J4.3 (Pin_3), U1.J2-12 (IO14)
- new net A4_B: J4.4 (Pin_4), U1.J3-16 (IO15)
- new net A4_IN_1: U6.3 (P12), U7.13 (BIN1)
- new net A4_IN_2: U6.4 (P13), U7.14 (BIN2)
- new net A4_OUT_1: J4.1 (Pin_1), U7.6 (BO1)
- new net A4_OUT_2: J4.2 (Pin_2), U7.7 (BO2)
- new net A4_PWM: U1.J3-8 (IO19), U7.15 (PWMB)
- no-connect marks 38 -> 30
Other:
- note removed: "Servo attachments"
- moved on the sheet: J13, J14, U2, U3

Commit message: 18-03-2026
Parts:
- removed D1: LED_RGBK, LED_THT:LED_D5.0mm-4_RGB_Staggered_Pins, symbol Library:LED_RGBK
- removed J8: Camera, Connector_JST:JST_XH_B2B-XH-A_1x02_P2.50mm_Vertical, symbol Library:Conn_01x02
- added D1: LED, LED_THT:LED_D3.0mm, symbol Device:LED
- added J10: Limit Switch 2, Connector_JST:JST_XH_B2B-XH-A_1x02_P2.50mm_Vertical, symbol Library:Conn_01x02
- added J8: Camera, Connector_JST:JST_XH_B4B-XH-A_1x04_P2.50mm_Vertical, symbol Library:Conn_01x04
- added J9: Limit Switch 1, Connector_JST:JST_XH_B2B-XH-A_1x02_P2.50mm_Vertical, symbol Library:Conn_01x02
- added R7: R, Resistor_THT:R_Axial_DIN0207_L6.3mm_D2.5mm_P7.62mm_Horizontal, symbol Library:R
- added SW3: SW_Push, Button_Switch_Keyboard:SW_Cherry_MX_1.00u_PCB, symbol Switch:SW_Push
Connections:
- net +3V3: now also J1.4 (Pin_4), J2.4 (Pin_4), J3.4 (Pin_4), J4.4 (Pin_4), J5.4 (Pin_4), J6.4 (Pin_4), U2.12 (STNDBY), U3.12 (STNDBY), U7.12 (STNDBY), J10.1 (Pin_1), J9.1 (Pin_1), SW3.1; no longer J1.5 (Pin_5), J2.5 (Pin_5), J3.5 (Pin_5), J4.5 (Pin_5), J5.5 (Pin_5), J6.5 (Pin_5)
- net +6V: now also J8.1 (Pin_1)
- net A1_A: now also J5.5 (Pin_5); no longer J5.3 (Pin_3)
- net A1_B: now also J5.6 (Pin_6); no longer J5.4 (Pin_4)
- net A2_A: now also J6.5 (Pin_5); no longer J6.3 (Pin_3)
- net A2_B: now also J6.6 (Pin_6); no longer J6.4 (Pin_4)
- net A3_A: now also J3.5 (Pin_5); no longer J3.3 (Pin_3)
- net A3_B: now also J3.6 (Pin_6); no longer J3.4 (Pin_4)
- net A4_A: now also J4.5 (Pin_5); no longer J4.3 (Pin_3)
- net A4_B: now also J4.6 (Pin_6); no longer J4.4 (Pin_4)
- net CAM_RX: now also J8.4 (Pin_4)
- net CAM_TX: now also J8.3 (Pin_3)
- net GND: now also J1.3 (Pin_3), J2.3 (Pin_3), J3.3 (Pin_3), J4.3 (Pin_3), J5.3 (Pin_3), J6.3 (Pin_3), D1.1 (K), J8.2 (Pin_2); no longer J1.6 (Pin_6), J2.6 (Pin_6), J3.6 (Pin_6), J4.6 (Pin_6), J5.6 (Pin_6), J6.6 (Pin_6)
- net L_A: now also J1.5 (Pin_5); no longer J1.3 (Pin_3)
- net L_B: now also J1.6 (Pin_6); no longer J1.4 (Pin_4)
- net R_A: now also J2.5 (Pin_5); no longer J2.3 (Pin_3)
- net R_B: now also J2.6 (Pin_6); no longer J2.4 (Pin_4)
- net LED_B renamed LIMIT_2
- net LIMIT_2: now also J10.2 (Pin_2)
- net LED_G renamed LIMIT_1
- net LIMIT_1: now also J9.2 (Pin_2)
- net LED_R renamed LED
- net LED: now also R7.1
- removed net STNDBY: U2.12 (STNDBY), U3.12 (STNDBY), U6.8 (P17), U7.12 (STNDBY)
- new net: D1.2 (A), R7.2
- new net BUTTON: SW3.2, U6.8 (P17)
Other:
- moved on the sheet: BZ1, J13, J14, J15, U4, U5

Commit message: Added sensors and state indication
Parts:
- U2, U3, U4, U5, U6, U7: value ~ -> (none)
